File: Design/DD_Power_1/DD_Power_1.kicad_pcb (KiCad board)
At the start: 2 copper layers, 110 x 47.8 mm, 94 parts, among them J1 POWER SUPPLY - 0349610340, U1 R-78HB5.0-0.5, U10 SN6505ADBV, U11 AZ1117H-ADJ, U12 SN6505ADBV, U13 AZ1117H-ADJ, U14 SN6505ADBV, U15 L7815, U2 NCV4276B, U3 AZ1117H-ADJ, U4 SN6505ADBV, U5 LM2596T-ADJ, U6 LM2596T-5, U7 AZ1117H-ADJ, U8 SN6505ADBV, U9 AZ1117H-ADJ

Commit message: Catchup commit.
Parts:
- removed C2: 100n, Capacitor_SMD:C_0805_2012Metric_Pad1.18x1.45mm_HandSolder
- removed U1: R-78HB5.0-0.5, Converter_DCDC:Converter_DCDC_RECOM_R-78HB-0.5_THT
- removed U2: NCV4276B, Package_TO_SOT_SMD:TO-263-5_TabPin3
- moved D13 0.10 mm to (212.6, 83.1)
Connections:
- J1 pad 10: +5V -> unconnected-(J1-Pad10)
- J1 pad 16: /+5VA_EN -> unconnected-(J1-Pad16)
- J1 pad 18: +5V -> unconnected-(J1-Pad18)
- J1 pad 19: +5VA -> unconnected-(J1-Pad19)
Routing:
- net /+12V_CONST: track 12.7 -> 0.00 mm
Other:
- copper layers 2 -> 4
