File: Design/DD_Power_2/DD_Power_2.kicad_pcb (KiCad board)
At the start: 2 copper layers, 110 x 47.8 mm, 94 parts, among them J1 POWER SUPPLY - 0349610340, U1 R-78HB5.0-0.5, U10 SN6505ADBV, U11 AZ1117H-ADJ, U12 SN6505ADBV, U13 AZ1117H-ADJ, U14 SN6505ADBV, U15 L7815, U2 NCV4276B, U3 AZ1117H-ADJ, U4 SN6505ADBV, U5 LM2596T-ADJ, U6 LM2596T-5, U7 AZ1117H-ADJ, U8 SN6505ADBV, U9 AZ1117H-ADJ

Commit message: Catchup commit.
Parts:
- removed the C10 at (237.2, 76.4)
- removed C21, C26, C36: 10uF, Capacitor_SMD:C_1206_3216Metric_Pad1.33x1.80mm_HandSolder
- removed C22, C27, C32, C37: C_Small, Capacitor_SMD:C_0805_2012Metric_Pad1.18x1.45mm_HandSolder
- removed C23, C25, C29, C30, C33, C34, C35, C38, C39, C40: 100nF, Capacitor_SMD:C_0805_2012Metric_Pad1.18x1.45mm_HandSolder
- removed the C31 at (192.2, 107.3)
- removed the C6 at (209.1, 97.2)
- removed the C7 at (206.0, 98.8)
- removed the C8 at (218.7, 90.0)
- removed the C9 at (237.2, 74.4)
- removed R10, R12, R14, R4, R8: 1k, Resistor_SMD:R_0805_2012Metric_Pad1.20x1.40mm_HandSolder
- removed R11, R13, R3, R7, R9: 4k7, Resistor_SMD:R_0805_2012Metric_Pad1.20x1.40mm_HandSolder
- removed TR1, TR2, TR3, TR4, TR5: Wuerth_750316031, Transformer_SMD:Transformer_Wuerth_750315371
- removed U1: R-78HB5.0-0.5, Converter_DCDC:Converter_DCDC_RECOM_R-78HB-0.5_THT
- removed U10, U12, U14, U4: SN6505ADBV, Package_TO_SOT_SMD:SOT-23-6
- removed U11, U13, U7, U9: AZ1117H-ADJ, Package_TO_SOT_SMD:SOT-223-3_TabPin2
- removed the U2 at (141.5, 88.0)
- removed the U3 at (205.9, 91.0)
- removed the U8 at (175.5, 103.2)
- added C16: 1uF, Capacitor_SMD:C_0805_2012Metric_Pad1.18x1.45mm_HandSolder, F.Cu at (198.9, 123.3)
- added C20: 1uF, Capacitor_SMD:C_0805_2012Metric_Pad1.18x1.45mm_HandSolder, F.Cu at (180.6, 134.9)
- added TP10: TestPoint, TestPoint:TestPoint_2Pads_Pitch2.54mm_Drill0.8mm, F.Cu at (180.0, 143.4)
- added TP2: TestPoint, TestPoint:TestPoint_2Pads_Pitch2.54mm_Drill0.8mm, F.Cu at (180.0, 120.1)
- added TP4: TestPoint, TestPoint:TestPoint_2Pads_Pitch2.54mm_Drill0.8mm, F.Cu at (198.3, 120.1)
- added TP6: TestPoint, TestPoint:TestPoint_2Pads_Pitch2.54mm_Drill0.8mm, F.Cu at (180.0, 131.8)
- added TP8: TestPoint, TestPoint:TestPoint_2Pads_Pitch2.54mm_Drill0.8mm, F.Cu at (198.3, 131.8)
- C2: value 100n -> 1uF
- C24, C28: value 100nF -> 1uF; moved to F.Cu
- moved C24 65.0 mm to (198.9, 134.9), turned to 0 degrees
- moved C2 62.5 mm to (180.6, 123.3)
- moved RV6 53.4 mm to (174.0, 145.0), turned to 0 degrees
- moved C28 50.1 mm to (180.6, 146.6)
- moved RV4 44.7 mm to (174.0, 133.4), turned to 0 degrees
- moved RV1 44.6 mm to (174.0, 121.7), turned to 0 degrees
- moved RV5 38.9 mm to (192.3, 133.4)
- moved RV3 31.7 mm to (192.3, 121.7), turned to 0 degrees
- renumbered C16 to C10, C17 to C11, C18 to C12, C19 to C13, C20 to C14, C41 to C31, C11 to C5, C12 to C6, C13 to C7, C14 to C8, C15 to C9, D3 to D1, D12 to D10, D13 to D11, D4 to D2, D5 to D3, D6 to D4, D7 to D5, D8 to D6, D9 to D7, D10 to D8, D11 to D9, TP2 to TP3, TP3 to TP5, TP4 to TP7, TP5 to TP9, U5 to U2, U6 to U3, U15 to U8
Connections:
- C24 pad 2: /FILAMENT_02A -> GND
- D6 pad 1: Net-(C24-Pad1) -> Net-(D6-Pad1)
- J1 pad 18: +5V -> unconnected-(J1-Pad18)
- J1 pad 19: +5VA -> unconnected-(J1-Pad19)
- RV1 pad 1: GND -> Net-(C4-Pad1)
- RV1 pad 2: Net-(R3-Pad1) -> Net-(C4-Pad1)
- RV1 pad 3: Net-(R3-Pad1) -> Net-(R2-Pad1)
- RV3 pad 1: GND -> Net-(C18-Pad1)
- RV3 pad 2: Net-(R7-Pad1) -> Net-(C18-Pad1)
- RV3 pad 3: Net-(R7-Pad1) -> Net-(R8-Pad1)
- RV4 pad 1: GND -> Net-(C22-Pad1)
- RV4 pad 2: Net-(R9-Pad1) -> Net-(C22-Pad1)
- RV4 pad 3: Net-(R9-Pad1) -> Net-(R12-Pad1)
- RV5 pad 1: GND -> Net-(C26-Pad1)
- RV5 pad 2: Net-(R11-Pad1) -> Net-(C26-Pad1)
- RV5 pad 3: Net-(R11-Pad1) -> Net-(R16-Pad1)
- RV6 pad 1: GND -> Net-(C30-Pad1)
- RV6 pad 2: Net-(R13-Pad1) -> Net-(C30-Pad1)
- RV6 pad 3: Net-(R13-Pad1) -> Net-(R20-Pad1)
- TP1 pad 1: Net-(C8-Pad1) -> /FILAMENT_01A
- TP3 pad 1: Net-(C23-Pad1) -> /FILAMENT_02B
- TP5 pad 1: Net-(C28-Pad1) -> /FILAMENT_03B
- TP7 pad 1: Net-(C33-Pad1) -> /FILAMENT_04B
- TP9 pad 1: Net-(C38-Pad1) -> /FILAMENT_05B
Routing:
- net /-22.5V_BIAS: track 4.31 -> 8.77 mm
- net Net-(C5-Pad1): track 31.4 -> 27.0 mm
- added copper zone on F.Cu, net Net-(D5-Pad1)
- removed copper zone on F.Cu, net Net-(D3-Pad1)
