File: Design/DD_Power_2/DD_Power_2.kicad_sch (KiCad schematic)
At the start: 12 parts, among them J1 POWER SUPPLY - 0349610340, U1 R-78HB5.0-0.5, U2 NCV4276B

Commit message: Catchup commit.
Parts:
- removed C1: 22uF, symbol Device:C_Polarized_Small
- removed C2: 100n, Capacitor_SMD:C_0805_2012Metric_Pad1.18x1.45mm_HandSolder, symbol Device:C_Small
- removed C3, C4: C_Small, symbol Device:C_Small
- removed C5: 22uF, symbol Device:C_Small
- removed D1: D_Small, symbol Device:D_Small
- removed D2: D_TVS, symbol Device:D_TVS
- removed R1, R2: R_Small, symbol Device:R_Small
- removed U1: R-78HB5.0-0.5, Converter_DCDC:Converter_DCDC_RECOM_R-78HB-0.5_THT, symbol Regulator_Switching:R-78HB5.0-0.5
- removed U2: NCV4276B, Package_TO_SOT_SMD:TO-263-5_TabPin3, symbol Personal:NCV4276B
Connections:
- net +5V: no longer J1.18 (Pin_18)
- net +5VA: no longer names the net of J1.19 (Pin_19)
