File: Design/DD_Power_2/Filament_Drive.kicad_sch (KiCad schematic)
At the start: 13 parts

Commit message: Catchup commit.
Parts:
- gave numbers to parts that had none: 11
- renumbered D3 to D1
Changed lines of the file:
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@@
   (symbol (lib_id "Device:D_Zener") (at 157.48 67.31 90) (mirror x)
     (in_bom yes) (on_board yes)
-    (property "Reference" "D3" (id 0) (at 159.512 68.4784 90)
+    (property "Reference" "D1" (id 0) (at 159.512 68.4784 90)
       (effects (font (size 1.27 1.27)) (justify right))
     )
@@
   (symbol (lib_id "power:GND") (at 118.11 62.23 0)
     (in_bom yes) (on_board yes) (fields_autoplaced)
-    (property "Reference" "#PWR026" (id 0) (at 118.11 68.58 0)
+    (property "Reference" "#PWR014" (id 0) (at 118.11 68.58 0)
       (effects (font (size 1.27 1.27)) hide)
     )
@@
   (symbol (lib_id "Device:C_Small") (at 77.47 45.72 90)
     (in_bom yes) (on_board yes) (fields_autoplaced)
-    (property "Reference" "C?" (id 0) (at 77.4763 39.37 90))
+    (property "Reference" "C1" (id 0) (at 77.4763 39.37 90))
     (property "Value" "C_Small" (id 1) (at 77.4763 41.91 90))
     (property "Footprint" "" (id 2) (at 77.47 45.72 0)
@@
   (symbol (lib_id "Personal:LM4871") (at 118.11 50.8 0)
     (in_bom yes) (on_board yes)
-    (property "Reference" "U?" (id 0) (at 119.38 39.37 0)
+    (property "Reference" "U1" (id 0) (at 119.38 39.37 0)
       (effects (font (size 1.27 1.27)) (justify left))
     )
@@
   (symbol (lib_id "Device:C_Small") (at 101.6 50.8 0)
     (in_bom yes) (on_board yes) (fields_autoplaced)
-    (property "Reference" "C?" (id 0) (at 104.14 49.5362 0)
+    (property "Reference" "C2" (id 0) (at 104.14 49.5362 0)
       (effects (font (size 1.27 1.27)) (justify left))
     )
@@
   (symbol (lib_id "Device:C_Small") (at 139.7 49.53 90)
     (in_bom yes) (on_board yes)
-    (property "Reference" "C?" (id 0) (at 139.7 44.45 90))
+    (property "Reference" "C4" (id 0) (at 139.7 44.45 90))
     (property "Value" "C_Small" (id 1) (at 139.7 46.99 90))
     (property "Footprint" "" (id 2) (at 139.7 49.53 0)
@@
   (symbol (lib_id "Device:R_Small") (at 109.22 27.94 270)
     (in_bom yes) (on_board yes)
-    (property "Reference" "R?" (id 0) (at 107.95 25.4 90)
+    (property "Reference" "R2" (id 0) (at 107.95 25.4 90)
       (effects (font (size 1.27 1.27)) (justify left))
     )
@@
   (symbol (lib_id "Connector:TestPoint") (at 146.05 52.07 180)
     (in_bom yes) (on_board yes)
-    (property "Reference" "TP?" (id 0) (at 144.78 55.88 0)
+    (property "Reference" "TP2" (id 0) (at 144.78 55.88 0)
       (effects (font (size 1.27 1.27)) (justify left))
     )
@@
   (symbol (lib_id "power:GND") (at 101.6 53.34 0)
     (in_bom yes) (on_board yes)
-    (property "Reference" "#PWR?" (id 0) (at 101.6 59.69 0)
+    (property "Reference" "#PWR013" (id 0) (at 101.6 59.69 0)
       (effects (font (size 1.27 1.27)) hide)
     )
@@
   (symbol (lib_id "Device:R_Small") (at 86.36 45.72 90)
     (in_bom yes) (on_board yes) (fields_autoplaced)
-    (property "Reference" "R?" (id 0) (at 86.36 39.37 90))
+    (property "Reference" "R1" (id 0) (at 86.36 39.37 90))
     (property "Value" "R_Small" (id 1) (at 86.36 41.91 90))
     (property "Footprint" "" (id 2) (at 86.36 45.72 0)
@@
   (symbol (lib_id "Device:R_Potentiometer_Small") (at 114.3 27.94 270)
     (in_bom yes) (on_board yes)
-    (property "Reference" "RV?" (id 0) (at 115.57 25.4 90)
+    (property "Reference" "RV1" (id 0) (at 115.57 25.4 90)
       (effects (font (size 1.27 1.27)) (justify right))
     )
@@
   (symbol (lib_id "Device:R_Small") (at 158.75 57.15 0)
     (in_bom yes) (on_board yes) (fields_autoplaced)
-    (property "Reference" "R?" (id 0) (at 161.29 55.8799 0)
+    (property "Reference" "R4" (id 0) (at 161.29 55.8799 0)
       (effects (font (size 1.27 1.27)) (justify left))
     )
@@
   (symbol (lib_id "Device:C_Small") (at 132.08 52.07 90)
     (in_bom yes) (on_board yes)
-    (property "Reference" "C?" (id 0) (at 132.08 57.15 90))
+    (property "Reference" "C3" (id 0) (at 132.08 57.15 90))
     (property "Value" "C_Small" (id 1) (at 132.08 54.61 90))
     (property "Footprint" "" (id 2) (at 132.08 52.07 0)
@@
   (symbol (lib_id "Device:R_Small") (at 156.21 57.15 0)
     (in_bom yes) (on_board yes)
-    (property "Reference" "R?" (id 0) (at 152.4 55.88 0)
-      (effects (font (size 1.27 1.27)) (justify left))
-    )
+    (property "Reference" "R3" (id 0) (at 152.4 55.88 0)
+      (effects (font (size 1.27 1.27)) (justify left))
+    )
