File: Design/DD_Power_2/Negative_Supply.kicad_sch (KiCad schematic)
At the start: 14 parts, among them U5 LM2596T-ADJ

Commit message: Catchup commit.
Parts:
- renumbered C16 to C10, C11 to C5, C12 to C6, C13 to C7, C14 to C8, C15 to C9, D4 to D2, D5 to D3, D6 to D4, U5 to U2
Changed lines of the file:
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@@
   (symbol (lib_id "Device:C_Polarized_Small") (at 142.24 92.71 0) (unit 1)
     (in_bom yes) (on_board yes) (fields_autoplaced)
-    (property "Reference" "C14" (id 0) (at 144.78 90.8938 0)
+    (property "Reference" "C8" (id 0) (at 144.78 90.8938 0)
       (effects (font (size 1.27 1.27)) (justify left))
     )
@@
   (symbol (lib_id "Regulator_Switching:LM2596T-ADJ") (at 114.3 86.36 0) (unit 1)
     (in_bom yes) (on_board yes) (fields_autoplaced)
-    (property "Reference" "U5" (id 0) (at 114.3 76.2 0))
+    (property "Reference" "U2" (id 0) (at 114.3 76.2 0))
     (property "Value" "LM2596T-ADJ" (id 1) (at 114.3 78.74 0))
     (property "Footprint" "Package_TO_SOT_THT:TO-220-5_P3.4x3.7mm_StaggerOdd_Lead3.8mm_Vertical" (id 2) (at 115.57 92.71 0)
@@
   (symbol (lib_id "Device:C_Polarized_Small") (at 60.96 87.63 0) (unit 1)
     (in_bom yes) (on_board yes) (fields_autoplaced)
-    (property "Reference" "C12" (id 0) (at 63.5 85.8138 0)
+    (property "Reference" "C6" (id 0) (at 63.5 85.8138 0)
       (effects (font (size 1.27 1.27)) (justify left))
     )
@@
   (symbol (lib_id "Device:D_Schottky_Small") (at 38.1 83.82 180) (unit 1)
     (in_bom yes) (on_board yes) (fields_autoplaced)
-    (property "Reference" "D4" (id 0) (at 38.354 77.47 0))
+    (property "Reference" "D2" (id 0) (at 38.354 77.47 0))
     (property "Value" "B540C-13-F" (id 1) (at 38.354 80.01 0))
     (property "Footprint" "Diode_SMD:D_SMC" (id 2) (at 38.1 83.82 90)
@@
   (symbol (lib_id "Device:C_Small") (at 171.45 73.66 0) (unit 1)
     (in_bom yes) (on_board yes) (fields_autoplaced)
-    (property "Reference" "C16" (id 0) (at 173.99 72.3962 0)
+    (property "Reference" "C10" (id 0) (at 173.99 72.3962 0)
       (effects (font (size 1.27 1.27)) (justify left))
     )
@@
   (symbol (lib_id "Device:C_Small") (at 157.48 92.71 0) (unit 1)
     (in_bom yes) (on_board yes) (fields_autoplaced)
-    (property "Reference" "C15" (id 0) (at 160.02 91.4462 0)
+    (property "Reference" "C9" (id 0) (at 160.02 91.4462 0)
       (effects (font (size 1.27 1.27)) (justify left))
     )
@@
   (symbol (lib_id "Device:C_Small") (at 76.2 87.63 0) (unit 1)
     (in_bom yes) (on_board yes) (fields_autoplaced)
-    (property "Reference" "C13" (id 0) (at 78.74 86.3662 0)
+    (property "Reference" "C7" (id 0) (at 78.74 86.3662 0)
       (effects (font (size 1.27 1.27)) (justify left))
     )
@@
   (symbol (lib_id "Device:D_Schottky_Small") (at 128.27 92.71 270) (unit 1)
     (in_bom yes) (on_board yes) (fields_autoplaced)
-    (property "Reference" "D5" (id 0) (at 130.81 91.1859 90)
+    (property "Reference" "D3" (id 0) (at 130.81 91.1859 90)
       (effects (font (size 1.27 1.27)) (justify left))
     )
@@
   (symbol (lib_id "power:GND") (at 44.45 90.17 0) (unit 1)
     (in_bom yes) (on_board yes)
-    (property "Reference" "#PWR028" (id 0) (at 44.45 96.52 0)
+    (property "Reference" "#PWR015" (id 0) (at 44.45 96.52 0)
       (effects (font (size 1.27 1.27)) hide)
     )
@@
   (symbol (lib_id "Device:C_Polarized_Small") (at 44.45 87.63 0) (unit 1)
     (in_bom yes) (on_board yes) (fields_autoplaced)
-    (property "Reference" "C11" (id 0) (at 46.99 85.8138 0)
+    (property "Reference" "C5" (id 0) (at 46.99 85.8138 0)
       (effects (font (size 1.27 1.27)) (justify left))
     )
@@
   (symbol (lib_id "Device:D_Small") (at 170.18 92.71 270) (unit 1)
     (in_bom yes) (on_board yes) (fields_autoplaced)
-    (property "Reference" "D6" (id 0) (at 172.72 91.4399 90)
-      (effects (font (size 1.27 1.27)) (justify left))
-    )
+    (property "Reference" "D4" (id 0) (at 172.72 91.4399 90)
+      (effects (font (size 1.27 1.27)) (justify left))
+    )
