File: Design/DD_Power_2/Positive_Supply.kicad_sch (KiCad schematic)
At the start: 7 parts, among them U6 LM2596T-5

Commit message: Catchup commit.
Parts:
- renumbered C17 to C11, C18 to C12, C19 to C13, C20 to C14, D7 to D5, U6 to U3
Changed lines of the file:
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@@
   (symbol (lib_id "Device:C_Small") (at 157.48 92.71 0) (unit 1)
     (in_bom yes) (on_board yes) (fields_autoplaced)
-    (property "Reference" "C20" (id 0) (at 160.02 91.4462 0)
+    (property "Reference" "C14" (id 0) (at 160.02 91.4462 0)
       (effects (font (size 1.27 1.27)) (justify left))
     )
@@
   (symbol (lib_id "Regulator_Switching:LM2596T-ADJ") (at 114.3 86.36 0) (unit 1)
     (in_bom yes) (on_board yes) (fields_autoplaced)
-    (property "Reference" "U6" (id 0) (at 114.3 76.2 0))
+    (property "Reference" "U3" (id 0) (at 114.3 76.2 0))
     (property "Value" "LM2596T-5" (id 1) (at 114.3 78.74 0))
     (property "Footprint" "Package_TO_SOT_THT:TO-220-5_P3.4x3.7mm_StaggerOdd_Lead3.8mm_Vertical" (id 2) (at 115.57 92.71 0)
@@
   (symbol (lib_id "power:GND") (at 44.45 100.33 0) (unit 1)
     (in_bom yes) (on_board yes)
-    (property "Reference" "#PWR029" (id 0) (at 44.45 106.68 0)
+    (property "Reference" "#PWR016" (id 0) (at 44.45 106.68 0)
       (effects (font (size 1.27 1.27)) hide)
     )
@@
   (symbol (lib_id "Device:D_Schottky_Small") (at 128.27 92.71 270) (unit 1)
     (in_bom yes) (on_board yes) (fields_autoplaced)
-    (property "Reference" "D7" (id 0) (at 130.81 91.1859 90)
+    (property "Reference" "D5" (id 0) (at 130.81 91.1859 90)
       (effects (font (size 1.27 1.27)) (justify left))
     )
@@
   (symbol (lib_id "Device:C_Small") (at 76.2 87.63 0) (unit 1)
     (in_bom yes) (on_board yes) (fields_autoplaced)
-    (property "Reference" "C18" (id 0) (at 78.74 86.3662 0)
+    (property "Reference" "C12" (id 0) (at 78.74 86.3662 0)
       (effects (font (size 1.27 1.27)) (justify left))
     )
@@
   (symbol (lib_id "Device:C_Polarized_Small") (at 44.45 87.63 0) (unit 1)
     (in_bom yes) (on_board yes) (fields_autoplaced)
-    (property "Reference" "C17" (id 0) (at 46.99 85.8138 0)
+    (property "Reference" "C11" (id 0) (at 46.99 85.8138 0)
       (effects (font (size 1.27 1.27)) (justify left))
     )
@@
   (symbol (lib_id "Device:C_Polarized_Small") (at 142.24 92.71 0) (unit 1)
     (in_bom yes) (on_board yes) (fields_autoplaced)
-    (property "Reference" "C19" (id 0) (at 144.78 90.8938 0)
+    (property "Reference" "C13" (id 0) (at 144.78 90.8938 0)
       (effects (font (size 1.27 1.27)) (justify left))
     )
