File: Design/DD_Power_2/Power_Input.kicad_sch (KiCad schematic)
At the start: 5 parts, among them U15 L7815

Commit message: Catchup commit.
Parts:
- renumbered C41 to C31, C42 to C32, D12 to D10, D13 to D11, U15 to U8
Changed lines of the file:
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@@
   (symbol (lib_id "Device:C_Polarized_Small") (at 95.25 73.66 0) (unit 1)
     (in_bom yes) (on_board yes)
-    (property "Reference" "C41" (id 0) (at 97.79 71.8438 0)
+    (property "Reference" "C31" (id 0) (at 97.79 71.8438 0)
       (effects (font (size 1.27 1.27)) (justify left))
     )
@@
   (symbol (lib_id "power:GND") (at 111.76 76.2 0) (unit 1)
     (in_bom yes) (on_board yes)
-    (property "Reference" "#PWR044" (id 0) (at 111.76 82.55 0)
+    (property "Reference" "#PWR027" (id 0) (at 111.76 82.55 0)
       (effects (font (size 1.27 1.27)) hide)
     )
@@
   (symbol (lib_id "Device:D_TVS") (at 85.09 74.93 90) (unit 1)
     (in_bom yes) (on_board yes) (fields_autoplaced)
-    (property "Reference" "D13" (id 0) (at 87.63 73.6599 90)
+    (property "Reference" "D11" (id 0) (at 87.63 73.6599 90)
       (effects (font (size 1.27 1.27)) (justify right))
     )
@@
   (symbol (lib_id "power:GND") (at 128.27 77.47 0) (unit 1)
     (in_bom yes) (on_board yes)
-    (property "Reference" "#PWR045" (id 0) (at 128.27 83.82 0)
+    (property "Reference" "#PWR028" (id 0) (at 128.27 83.82 0)
       (effects (font (size 1.27 1.27)) hide)
     )
@@
   (symbol (lib_id "Device:D_Dual_CommonCathode_AKA") (at 73.66 69.85 90) (unit 1)
     (in_bom yes) (on_board yes) (fields_autoplaced)
-    (property "Reference" "D12" (id 0) (at 71.12 68.5799 90)
+    (property "Reference" "D10" (id 0) (at 71.12 68.5799 90)
       (effects (font (size 1.27 1.27)) (justify left))
     )
@@
   (symbol (lib_id "power:GND") (at 85.09 78.74 0) (unit 1)
     (in_bom yes) (on_board yes)
-    (property "Reference" "#PWR042" (id 0) (at 85.09 85.09 0)
+    (property "Reference" "#PWR025" (id 0) (at 85.09 85.09 0)
       (effects (font (size 1.27 1.27)) hide)
     )
@@
   (symbol (lib_id "Regulator_Linear:L7815") (at 128.27 69.85 0) (unit 1)
     (in_bom yes) (on_board yes) (fields_autoplaced)
-    (property "Reference" "U15" (id 0) (at 128.27 62.23 0))
+    (property "Reference" "U8" (id 0) (at 128.27 62.23 0))
     (property "Value" "L7815" (id 1) (at 128.27 64.77 0))
     (property "Footprint" "Package_TO_SOT_THT:TO-220-3_Vertical" (id 2) (at 128.905 73.66 0)
@@
   (symbol (lib_id "power:GND") (at 95.25 76.2 0) (unit 1)
     (in_bom yes) (on_board yes)
-    (property "Reference" "#PWR043" (id 0) (at 95.25 82.55 0)
+    (property "Reference" "#PWR026" (id 0) (at 95.25 82.55 0)
       (effects (font (size 1.27 1.27)) hide)
     )
@@
   (symbol (lib_id "Device:C_Small") (at 111.76 73.66 0) (unit 1)
     (in_bom yes) (on_board yes) (fields_autoplaced)
-    (property "Reference" "C42" (id 0) (at 114.3 72.3962 0)
+    (property "Reference" "C32" (id 0) (at 114.3 72.3962 0)
       (effects (font (size 1.27 1.27)) (justify left))
     )
