File: Design/DD_Warning_Module_1/DD_Warning_Module_1.kicad_pcb (KiCad board)
At the start: 2 copper layers, 324.6 x 35 mm, 29 parts, among them J1 Conn_01x04, J2 BL_3

Commit message: warning module update; ws2812->ws2813 (backup data in)
Parts:
- C1, C13, C2, C3, R1: moved to F.Cu
- D10, D11, D4, D5, D6, D7, D8, D9: value SK6812 -> WS2813; footprint LED_SMD:LED_SK6812_PLCC4_5.0x5.0mm_P3.2mm -> LED_SMD:LED_WS2812_PLCC6_5.0x5.0mm_P1.6mm
- D12: value Turn_R -> WS2813; footprint LED_THT:LED_D5.0mm-4_RGB -> LED_SMD:LED_WS2812_PLCC6_5.0x5.0mm_P1.6mm
- D3: value Turn_L -> WS2813; footprint LED_THT:LED_D5.0mm-4_RGB -> LED_SMD:LED_WS2812_PLCC6_5.0x5.0mm_P1.6mm
- moved C3 7.30 mm to (89.0, 115.9), turned to 0 degrees
- moved C2 5.56 mm to (336.4, 117.5)
- moved C13 5.45 mm to (278.5, 115.7), turned to 0 degrees
- moved C1 5.03 mm to (23.1, 116.8)
- moved D2 3.23 mm to (27.3, 115.3), turned to -90 degrees
- moved D1 3.08 mm to (332.0, 115.6), turned to -90 degrees
- moved D12 2.94 mm to (273.1, 114.1)
- moved D3 2.42 mm to (83.6, 114.2)
Connections:
- D1 pad 4: Net-(D1-Pad4) -> Net-(D1-DIN)
- D10 pad 1: GND -> +5V
- D10 pad 2: Net-(D10-Pad2) -> +5V
- D10 pad 3: +5V -> Net-(D10-DOUT)
- D10 pad 4: Net-(D10-Pad4) -> Net-(D10-DIN)
- D11 pad 1: GND -> +5V
- D11 pad 2: Net-(D10-Pad4) -> +5V
- D11 pad 3: +5V -> Net-(D11-DOUT)
- D11 pad 4: Net-(D11-Pad4) -> Net-(D10-DOUT)
- D12 pad 1: Net-(D12-Pad1) -> +5V
- D12 pad 2: GND -> +5V
- D12 pad 3: +5V -> Net-(D12-DOUT)
- D12 pad 4: Net-(D11-Pad4) -> Net-(D11-DOUT)
- D2 pad 1: Net-(D2-Pad1) -> Net-(D2-DOUT)
- D2 pad 4: Net-(D1-Pad4) -> Net-(D1-DIN)
- D3 pad 1: Net-(D3-Pad1) -> +5V
- D3 pad 2: GND -> +5V
- D3 pad 3: +5V -> Net-(D3-DOUT)
- D3 pad 4: Net-(D2-Pad1) -> Net-(D2-DOUT)
- D4 pad 1: GND -> +5V
- D4 pad 2: Net-(D3-Pad1) -> +5V
- D4 pad 3: +5V -> Net-(D4-DOUT)
- D4 pad 4: Net-(D4-Pad4) -> Net-(D3-DOUT)
- D5 pad 1: GND -> +5V
- D5 pad 2: Net-(D4-Pad4) -> +5V
- D5 pad 3: +5V -> Net-(D5-DOUT)
- D5 pad 4: Net-(D5-Pad4) -> Net-(D4-DOUT)
- D6 pad 1: GND -> +5V
- D6 pad 2: Net-(D5-Pad4) -> +5V
- D6 pad 3: +5V -> Net-(D6-DOUT)
- D6 pad 4: Net-(D6-Pad4) -> Net-(D5-DOUT)
- D7 pad 1: GND -> +5V
- D7 pad 2: Net-(D6-Pad4) -> +5V
- D7 pad 3: +5V -> Net-(D7-DOUT)
- D7 pad 4: Net-(D7-Pad4) -> Net-(D6-DOUT)
- D8 pad 1: GND -> +5V
- D8 pad 2: Net-(D7-Pad4) -> +5V
- D8 pad 3: +5V -> Net-(D10-BIN)
- D8 pad 4: Net-(D8-Pad4) -> Net-(D7-DOUT)
- D9 pad 1: GND -> +5V
- D9 pad 2: Net-(D8-Pad4) -> +5V
- D9 pad 3: +5V -> Net-(D10-DIN)
- D9 pad 4: Net-(D10-Pad2) -> Net-(D10-BIN)
- J1 pad 3: Net-(D12-Pad1) -> Net-(D12-DOUT)
- J2 pad 2: Net-(D1-Pad4) -> Net-(D1-DIN)
- R1 pad 2: Net-(D1-Pad4) -> Net-(D1-DIN)
Routing:
- net Net-(D1-DIN): track 0.00 -> 387.1 mm
- net Net-(D1-Pad4): track 386.0 -> 0.00 mm, vias 1 -> 0
- net Net-(D12-Pad1): track 186.8 -> 0.00 mm
- net Net-(D12-DOUT): track 0.00 -> 186.6 mm
- net Net-(D2-DOUT): track 0.00 -> 92.1 mm, vias 0 -> 4
- net Net-(D2-Pad1): track 64.2 -> 0.00 mm
- net GND: track 47.3 -> 0.00 mm, vias 82 -> 91
- net Net-(D3-DOUT): track 0.00 -> 42.7 mm, vias 0 -> 2
- net Net-(D10-DOUT): track 0.00 -> 41.1 mm, vias 0 -> 2
- net Net-(D4-DOUT): track 0.00 -> 39.5 mm, vias 0 -> 2
- net Net-(D5-DOUT): track 0.00 -> 39.2 mm, vias 0 -> 2
- net Net-(D7-DOUT): track 0.00 -> 38.8 mm, vias 0 -> 2
- net Net-(D10-DIN): track 0.00 -> 38.7 mm, vias 0 -> 2
- net Net-(D10-BIN): track 0.00 -> 38.5 mm, vias 0 -> 2
- net Net-(D6-DOUT): track 0.00 -> 38.4 mm, vias 0 -> 2
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